File: lets_split.kicad_pcb (KiCad board)
At the start: 2 copper layers, 111.8 x 79 mm, 67 parts, among them J1 3PIN, J2 6PIN, J3 3PIN, J4 3PIN, J5 3PIN, M1 FIDUCIAL, M2 FIDUCIAL, M3 FIDUCIAL, M4 FIDUCIAL, SW1 SW_PUSH, SW10 SW_PUSH, SW11 SW_PUSH, SW12 SW_PUSH, SW13 SW_PUSH, SW14 SW_PUSH, SW15 SW_PUSH, SW16 SW_PUSH, SW17 SW_PUSH, SW18 SW_PUSH, SW19 SW_PUSH, SW2 SW_PUSH, SW20 SW_PUSH, SW21 SW_PUSH, SW22 SW_PUSH, SW23 SW_PUSH, SW24 SW_PUSH, SW3 SW_PUSH, SW4 SW_PUSH, SW5 SW_PUSH, SW6 SW_PUSH, SW7 SW_PUSH, SW8 SW_PUSH, SW9 SW_PUSH, U1 ProMicro, U2 HOLE, U3 HOLE, U4 HOLE, U5 HOLE

Commit message: Use local holes and JUMPER_SMD_2DUB
Parts:
- U2, U3, U4: footprint prettylib:HOLE -> local:HOLE
- U5: footprint prettylib:HOLE -> local:HOLE_2
- W1: footprint prettylib:JUMPER_SMD_2DUB -> local:JUMPER_SMD_2DUB
